Commit message: updating urdf file and more accurate wheel_odom measurements

File: pi/daro_ros2_ws/src/daro_description/urdf/daro_min.urdf (robot description, URDF)
Before this commit: robot daro_min, 2 links, 1 joints
Links:
- added link caster_wheel; collision sphere radius=0.0127; visual sphere radius=0.0127
- added link left_wheel; collision cylinder length=0.025 radius=0.045; visual cylinder length=0.025 radius=0.045
- added link right_wheel; collision cylinder length=0.025 radius=0.045; visual cylinder length=0.025 radius=0.045
- link base_link: geometry collision box size=0.2223 0.1969 0.0254; visual box size=0.2223 0.1969 0.0254
Joints:
- added joint caster_joint: type fixed, parent base_link, child caster_wheel, origin xyz=0.1112 0 0.0127 rpy=0 0 0
- added joint left_wheel_joint: type continuous, parent base_link, child left_wheel, origin xyz=-0.0730 0.1207 0.045 rpy=0 0 0, axis 0 1 0
- added joint right_wheel_joint: type continuous, parent base_link, child right_wheel, origin xyz=-0.0730 -0.1207 0.045 rpy=0 0 0, axis 0 1 0
- joint laser_joint: origin xyz=0.08 0 0.10 rpy=0 0 0 -> xyz=-0.0730 0 0.0406 rpy=0 0 0
